File: Hardware/Spanner/Spanner/Spanner.kicad_pcb (KiCad board)
At the start: 2 copper layers, 59.8 x 55.2 mm, 69 parts, among them J1 USB_B_Micro, J2 SWD, J3 MOTOR, J4 MOTOR, J5 MOTOR, J6 Conn_01x05_Male, J7 Conn_01x02_Male, J8 MOTOR, Q1 BC846, Q3 BC846, Q5 BC846, Q6 BC846, U1 STM32L412K8Tx, U2 USBLC6-2SC6, U3 CURRENT_SENS, U4 RFM95W-868S2, U5 MCP1812BT_033TT, U6 OPA990

Commit message: Update various modules
Parts:
- removed J7: Conn_01x02_Male, Connector_PinHeader_2.54mm:PinHeader_1x02_P2.54mm_Vertical
- added D7: SD0603, Diode_SMD:D_0603_1608Metric, F.Cu at (114.5, 124.5)
- U5: value MCP1812BT_033TT -> MCP1812AT-033/TT
Connections:
- net DI_IN_2 renamed SW_EXT
Routing:
- net +5V: track 118.0 -> 108.7 mm
- net VBUS: track 14.8 -> 23.1 mm, vias 0 -> 1
- net GND: track 105.6 -> 101.2 mm
- net Net-(C3-Pad1): track 4.46 -> 5.96 mm

Commit message: update spanner
Connections:
- U1 pad 15: PWM_2 -> VUSB
- U1 pad 26: VUSB -> PWM_2
- U4 pad 2: SPI_MOSI -> SPI_MISO
- U4 pad 3: SPI_MISO -> SPI_MOSI
Routing:
- net VUSB: track 13.2 -> 23.4 mm, vias 0 -> 2
- net SPI_MISO: track 6.47 -> 12.5 mm, vias 0 -> 2
- net PWM_2: track 22.3 -> 28.0 mm
- net SPI_MOSI: track 7.26 -> 5.70 mm
- net PWM_1: track 37.3 -> 36.7 mm

Commit message: FW update
Parts:
- removed R21: 10k, Resistor_SMD:R_0603_1608Metric
Routing:
- net +24V: track 25.0 -> 22.0 mm
Changed lines of the file:
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@@
-    )
-  )
-  (footprint "Resistor_SMD:R_0603_1608Metric" (layer "F.Cu")
-    (at 109 97.5 180)
-    (descr "Resistor SMD 0603 (1608 Metric), square (rectangular) end terminal, IPC_7351 nominal, (Body size source: IPC-SM-782 page 72, https://www.pcb-3d.com/wordpress/wp-content/uploads/ipc-sm-782a_amendment_1_and_2.pdf), generated with kicad-footprint-generator")
-    (tags "resistor")
-    (property "Hersteller Nr." "RT0603FRE0710KL")
-    (property "Mouser Nr." "603-RT0603FRE0710KL")
-    (property "Sheetfile" "Main.kicad_sch")
-    (property "Sheetname" "Main")
-    (attr smd)
-    (fp_text reference "R21" (at 0 -1.43) (layer "F.SilkS")
-      (effects (font (size 1 1) (thickness 0.15)))
-    )
-    (fp_text value "10k" (at 0 1.43) (layer "F.Fab")
-      (effects (font (size 1 1) (thickness 0.15)))
-    )
-    (fp_text user "${REFERENCE}" (at 0 0) (layer "F.Fab")
-      (effects (font (size 0.4 0.4) (thickness 0.06)))
-    )
-    (fp_line (start -0.237258 -0.5225) (end 0.237258 -0.5225) (layer "F.SilkS") (width 0.12))
-    (fp_line (start -0.237258 0.5225) (end 0.237258 0.5225) (layer "F.SilkS") (width 0.12))
-    (fp_line (start 1.48 0.73) (end -1.48 0.73) (layer "F.CrtYd") (width 0.05))
-    (fp_line (start 1.48 -0.73) (end 1.48 0.73) (layer "F.CrtYd") (width 0.05))
-    (fp_line (start -1.48 -0.73) (end 1.48 -0.73) (layer "F.CrtYd") (width 0.05))
-    (fp_line (start -1.48 0.73) (end -1.48 -0.73) (layer "F.CrtYd") (width 0.05))
-    (fp_line (start 0.8 -0.4125) (end 0.8 0.4125) (layer "F.Fab") (width 0.1))
-    (fp_line (start 0.8 0.4125) (end -0.8 0.4125) (layer "F.Fab") (width 0.1))
-    (fp_line (start -0.8 0.4125) (end -0.8 -0.4125) (layer "F.Fab") (width 0.1))
-    (fp_line (start -0.8 -0.4125) (end 0.8 -0.4125) (layer "F.Fab") (width 0.1))
-    (pad "1" smd roundrect (at -0.825 0 180) (size 0.8 0.95) (layers "F.Cu" "F.Paste" "F.Mask") (roundrect_rratio 0.25)
-      (net 21 "+24V") (pintype "passive"))
-    (pad "2" smd roundrect (at 0.825 0 180) (size 0.8 0.95) (layers "F.Cu" "F.Paste" "F.Mask") (roundrect_rratio 0.25)
-      (net 50 "POWER_FET_OUT") (pintype "passive"))
-    (model "${KICAD6_3DMODEL_DIR}/Resistor_SMD.3dshapes/R_0603_1608Metric.wrl"
-      (offset (xyz 0 0 0))
-      (scale (xyz 1 1 1))
-      (rotate (xyz 0 0 0))
     )
   )
@@
   (segment (start 87.75 126.75) (end 87.25 126.25) (width 0.25) (layer "F.Cu") (net 20))
   (segment (start 85.4375 124.9375) (end 85.4375 124.25) (width 0.25) (layer "F.Cu") (net 20))
+  (segment (start 111.175 97.5) (end 111.175 98.158534) (width 0.25) (layer "F.Cu") (net 21))
   (segment (start 116.675 105.25) (end 115.6245 105.25) (width 0.25) (layer "F.Cu") (net 21))
+  (segment (start 111.508233 98.491767) (end 116.508233 98.491767) (width 0.25) (layer "F.Cu") (net 21))
   (segment (start 118.25 100.75) (end 118.25 99.863604) (width 0.25) (layer "F.Cu") (net 21))
-  (segment (start 109.825 97.5) (end 111.425 97.5) (width 0.25) (layer "F.Cu") (net 21))
-  (segment (start 109.991767 98.491767) (end 116.508233 98.491767) (width 0.25) (layer "F.Cu") (net 21))
   (segment (start 118.5 101) (end 118.25 100.75) (width 0.25) (layer "F.Cu") (net 21))
   (segment (start 121 101) (end 118.5 101) (width 0.25) (layer "F.Cu") (net 21))
-  (segment (start 109.825 97.5) (end 109.825 98.325) (width 0.25) (layer "F.Cu") (net 21))
   (segment (start 116.878163 98.491767) (end 116.508233 98.491767) (width 0.25) (layer "F.Cu") (net 21))
   (segment (start 118.25 99.863604) (end 116.878163 98.491767) (width 0.25) (layer "F.Cu") (net 21))
-  (segment (start 109.825 98.325) (end 109.991767 98.491767) (width 0.25) (layer "F.Cu") (net 21))
+  (segment (start 111.175 98.158534) (end 111.508233 98.491767) (width 0.25) (layer "F.Cu") (net 21))
   (via (at 115.6245 105.25) (size 0.6) (drill 0.3) (layers "F.Cu" "B.Cu") (net 21))
   (segment (start 118.25 101) (end 117.5 101.75) (width 0.25) (layer "B.Cu") (net 21))
@@
   (segment (start 108.3 104.075) (end 108.3 102.7) (width 0.25) (layer "F.Cu") (net 49))
   (segment (start 110.45 102.3) (end 110.75 102) (width 0.25) (layer "F.Cu") (net 49))
-  (segment (start 106.825 97.5) (end 108.175 97.5) (width 0.25) (layer "F.Cu") (net 50))
+  (segment (start 106.825 97.5) (end 107.75 97.5) (width 0.25) (layer "F.Cu") (net 50))
+  (segment (start 107.75 97.5) (end 108.175 97.925) (width 0.25) (layer "F.Cu") (net 50))
   (segment (start 119.79 103.54) (end 121 103.54) (width 0.25) (layer "F.Cu") (net 50))
   (segment (start 119.79 103.54) (end 117.75 101.5) (width 0.25) (layer "F.Cu") (net 50))
   (segment (start 117.75 100) (end 116.691767 98.941767) (width 0.25) (layer "F.Cu") (net 50))
-  (segment (start 108.175 98.675) (end 108.175 97.5) (width 0.25) (layer "F.Cu") (net 50))
   (segment (start 117.75 101.5) (end 117.75 100) (width 0.25) (layer "F.Cu") (net 50))
+  (segment (start 108.175 98.675) (end 108.175 97.925) (width 0.25) (layer "F.Cu") (net 50))
   (segment (start 108.441767 98.941767) (end 108.175 98.675) (width 0.25) (layer "F.Cu") (net 50))
   (segment (start 116.691767 98.941767) (end 108.441767 98.941767) (width 0.25) (layer "F.Cu") (net 50))
