File: Hardware/Spanner/Spanner/Spanner.kicad_sch (KiCad schematic)
At the start: 0 parts

Commit message: FW update
Parts:
- added D8: D, symbol Device:D
- added Q2: POWER_PMOS, symbol Device:Q_PMOS_DSG
- added R21: 1K, symbol Device:R
- added SW1: SW, symbol Switch:SW_MEC_5G
Connections:
- new net +24V: D8.1 (K), Q2.1 (D)
- new net EXT_SW_INPUT: D8.2 (A), SW1.1 (A), SW1.2 (A)
- new net POWER_FET_OUT: Q2.3 (G), R21.2
- new net VPP: Q2.2 (S), R21.1, SW1.3 (B), SW1.4 (B)
Other:
- note added: "external components"
Changed lines of the file:
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@@
 (kicad_sch (version 20211123) (generator eeschema)
   (paper "A4")
+  (junction (at 67.31 137.16) (diameter 0) (color 0 0 0 0)
+  )
+  (junction (at 66.04 115.57) (diameter 0) (color 0 0 0 0)
+  )
+  (junction (at 52.07 125.73) (diameter 0) (color 0 0 0 0)
+  )
+  (junction (at 81.28 115.57) (diameter 0) (color 0 0 0 0)
+  )
+  (junction (at 81.28 125.73) (diameter 0) (color 0 0 0 0)
+  )
+  (wire (pts (xy 60.96 105.41) (xy 66.04 105.41))
+    (stroke (width 0) (type default) (color 0 0 0 0))
+  )
+  (wire (pts (xy 81.28 128.27) (xy 81.28 125.73))
+    (stroke (width 0) (type default) (color 0 0 0 0))
+  )
+  (wire (pts (xy 44.45 125.73) (xy 52.07 125.73))
+    (stroke (width 0) (type default) (color 0 0 0 0))
+  )
+  (wire (pts (xy 66.04 115.57) (xy 67.31 115.57))
+    (stroke (width 0) (type default) (color 0 0 0 0))
+  )
+  (wire (pts (xy 81.28 111.76) (xy 81.28 115.57))
+    (stroke (width 0) (type default) (color 0 0 0 0))
+  )
+  (wire (pts (xy 44.45 125.73) (xy 44.45 123.19))
+    (stroke (width 0) (type default) (color 0 0 0 0))
+  )
+  (wire (pts (xy 63.5 115.57) (xy 66.04 115.57))
+    (stroke (width 0) (type default) (color 0 0 0 0))
+  )
+  (wire (pts (xy 67.31 133.35) (xy 67.31 137.16))
+    (stroke (width 0) (type default) (color 0 0 0 0))
+  )
+  (wire (pts (xy 81.28 135.89) (xy 81.28 137.16))
+    (stroke (width 0) (type default) (color 0 0 0 0))
+  )
+  (wire (pts (xy 66.04 105.41) (xy 66.04 115.57))
+    (stroke (width 0) (type default) (color 0 0 0 0))
+  )
+  (wire (pts (xy 63.5 137.16) (xy 67.31 137.16))
+    (stroke (width 0) (type default) (color 0 0 0 0))
+  )
+  (wire (pts (xy 81.28 115.57) (xy 81.28 125.73))
+    (stroke (width 0) (type default) (color 0 0 0 0))
+  )
+  (wire (pts (xy 52.07 115.57) (xy 52.07 125.73))
+    (stroke (width 0) (type default) (color 0 0 0 0))
+  )
+  (wire (pts (xy 77.47 115.57) (xy 81.28 115.57))
+    (stroke (width 0) (type default) (color 0 0 0 0))
+  )
+  (wire (pts (xy 52.07 125.73) (xy 62.23 125.73))
+    (stroke (width 0) (type default) (color 0 0 0 0))
+  )
+  (wire (pts (xy 55.88 115.57) (xy 52.07 115.57))
+    (stroke (width 0) (type default) (color 0 0 0 0))
+  )
+  (wire (pts (xy 67.31 137.16) (xy 81.28 137.16))
+    (stroke (width 0) (type default) (color 0 0 0 0))
+  )
+  (wire (pts (xy 81.28 125.73) (xy 72.39 125.73))
+    (stroke (width 0) (type default) (color 0 0 0 0))
+  )
+  (text "external components\n" (at 39.37 100.33 0)
+    (effects (font (size 1.27 1.27)) (justify left bottom))
+  )
+  (global_label "POWER_FET_OUT" (shape input) (at 63.5 137.16 180) (fields_autoplaced)
+    (effects (font (size 1.27 1.27)) (justify right))
+    (property "Intersheet References" "${INTERSHEET_REFS}" (id 0) (at 45.8469 137.2394 0)
+      (effects (font (size 1.27 1.27)) (justify right) hide)
+    )
+  )
+  (global_label "EXT_SW_INPUT" (shape input) (at 60.96 105.41 180) (fields_autoplaced)
+    (effects (font (size 1.27 1.27)) (justify right))
+    (property "Intersheet References" "${INTERSHEET_REFS}" (id 0) (at 45.1212 105.3306 0)
+      (effects (font (size 1.27 1.27)) (justify right) hide)
+    )
+  )
+  (symbol (lib_id "Device:D") (at 59.69 115.57 0) (unit 1)
+    (in_bom yes) (on_board yes) (fields_autoplaced)
+    (property "Reference" "D8" (id 0) (at 59.69 109.22 0))
+    (property "Value" "D" (id 1) (at 59.69 111.76 0))
+    (property "Footprint" "" (id 2) (at 59.69 115.57 0)
+      (effects (font (size 1.27 1.27)) hide)
+    )
+    (property "Datasheet" "~" (id 3) (at 59.69 115.57 0)
+      (effects (font (size 1.27 1.27)) hide)
+    )
+    (pin "1")
+    (pin "2")
+  )
+  (symbol (lib_id "power:VPP") (at 81.28 111.76 0) (unit 1)
+    (in_bom yes) (on_board yes) (fields_autoplaced)
+    (property "Reference" "#PWR0133" (id 0) (at 81.28 115.57 0)
+      (effects (font (size 1.27 1.27)) hide)
+    )
+    (property "Value" "VPP" (id 1) (at 81.28 106.68 0))
+    (property "Footprint" "" (id 2) (at 81.28 111.76 0)
+      (effects (font (size 1.27 1.27)) hide)
+    )
+    (property "Datasheet" "" (id 3) (at 81.28 111.76 0)
+      (effects (font (size 1.27 1.27)) hide)
+    )
+    (pin "1")
+  )
+  (symbol (lib_id "Switch:SW_MEC_5G") (at 72.39 115.57 0) (unit 1)
+    (in_bom yes) (on_board yes) (fields_autoplaced)
+    (property "Reference" "SW1" (id 0) (at 72.39 107.95 0))
+    (property "Value" "SW" (id 1) (at 72.39 110.49 0))
+    (property "Footprint" "" (id 2) (at 72.39 110.49 0)
+      (effects (font (size 1.27 1.27)) hide)
+    )
+    (property "Datasheet" "http://www.apem.com/int/index.php?controller=attachment&id_attachment=488" (id 3) (at 72.39 110.49 0)
+      (effects (font (size 1.27 1.27)) hide)
+    )
+    (pin "1")
+    (pin "3")
+    (pin "2")
+    (pin "4")
+  )
+  (symbol (lib_id "power:+24V") (at 44.45 123.19 0) (unit 1)
+    (in_bom yes) (on_board yes) (fields_autoplaced)
+    (property "Reference" "#PWR0150" (id 0) (at 44.45 127 0)
+      (effects (font (size 1.27 1.27)) hide)
+    )
+    (property "Value" "+24V" (id 1) (at 44.45 118.11 0))
+    (property "Footprint" "" (id 2) (at 44.45 123.19 0)
+      (effects (font (size 1.27 1.27)) hide)
+    )
+    (property "Datasheet" "" (id 3) (at 44.45 123.19 0)
+      (effects (font (size 1.27 1.27)) hide)
+    )
+    (pin "1")
+  )
+  (symbol (lib_id "Device:R") (at 81.28 132.08 0) (unit 1)
+    (in_bom yes) (on_board yes) (fields_autoplaced)
+    (property "Reference" "R21" (id 0) (at 83.82 130.8099 0)
+      (effects (font (size 1.27 1.27)) (justify left))
+    )
+    (property "Value" "1K" (id 1) (at 83.82 133.3499 0)
+      (effects (font (size 1.27 1.27)) (justify left))
+    )
+    (property "Footprint" "" (id 2) (at 79.502 132.08 90)
+      (effects (font (size 1.27 1.27)) hide)
+    )
+    (property "Datasheet" "~" (id 3) (at 81.28 132.08 0)
+      (effects (font (size 1.27 1.27)) hide)
+    )
+    (pin "1")
+    (pin "2")
+  )
+  (symbol (lib_id "Device:Q_PMOS_DSG") (at 67.31 128.27 90) (unit 1)
+    (in_bom yes) (on_board yes)
+    (property "Reference" "Q2" (id 0) (at 67.31 119.38 90))
+    (property "Value" "POWER_PMOS" (id 1) (at 67.31 121.92 90))
+    (property "Footprint" "" (id 2) (at 64.77 123.19 0)
+      (effects (font (size 1.27 1.27)) hide)
+    )
+    (property "Datasheet" "~" (id 3) (at 67.31 128.27 0)
+      (effects (font (size 1.27 1.27)) hide)
+    )
+    (pin "1")
+    (pin "2")
+    (pin "3")
+  )
   (sheet (at 112.395 23.495) (size 82.55 44.45) (fields_autoplaced)
     (stroke (width 0.1524) (type solid) (color 0 0 0 0))
@@
       (reference "#PWR0132") (unit 1) (value "GND") (footprint "")
     )
+    (path "/71ddd14d-eb3d-43a6-84d1-7511bb2698f5"
+      (reference "#PWR0133") (unit 1) (value "VPP") (footprint "")
+    )
     (path "/cb73e00e-b752-4474-a136-20146bf8e401/1d68dfd5-05b1-42b5-b5cc-d78800ff7fc8"
       (reference "#PWR0134") (unit 1) (value "GND") (footprint "")
@@
       (reference "#PWR0149") (unit 1) (value "GND") (footprint "")
     )
-    (path "/cb73e00e-b752-4474-a136-20146bf8e401/46bc8aa0-6f74-4edf-af50-35d408afc3da"
+    (path "/9776ec40-aae8-465c-82cc-0e6702af69d4"
       (reference "#PWR0150") (unit 1) (value "+24V") (footprint "")
     )
@@
       (reference "D7") (unit 1) (value "SD0603") (footprint "Diode_SMD:D_0603_1608Metric")
     )
+    (path "/3a6520c7-ad5c-4751-9ad3-c78f2aa87c9f"
+      (reference "D8") (unit 1) (value "D") (footprint "")
+    )
     (path "/cb73e00e-b752-4474-a136-20146bf8e401/0c3f4d7d-96f3-42f5-b1aa-653f0fe5929b"
       (reference "H1") (unit 1) (value "MountingHole") (footprint "MountingHole:MountingHole_3.2mm_M3")
@@
       (reference "Q1") (unit 1) (value "BC846") (footprint "Package_TO_SOT_SMD:SOT-23")
     )
+    (path "/d7bcc113-c39f-4864-bf3a-a328b6fe5780"
+      (reference "Q2") (unit 1) (value "POWER_PMOS") (footprint "")
+    )
     (path "/cb73e00e-b752-4474-a136-20146bf8e401/c5b98b84-6d99-4f5d-993c-6e83074bcdba"
       (reference "Q3") (unit 1) (value "BC846") (footprint "Package_TO_SOT_SMD:SOT-23")
@@
       (reference "R20") (unit 1) (value "1k") (footprint "Resistor_SMD:R_0603_1608Metric")
     )
-    (path "/cb73e00e-b752-4474-a136-20146bf8e401/5d8060b5-145a-492e-95f6-5c00f6d72938"
-      (reference "R21") (unit 1) (value "10k") (footprint "Resistor_SMD:R_0603_1608Metric")
+    (path "/97c939b4-9e79-476e-875c-1c48dcc85614"
+      (reference "R21") (unit 1) (value "1K") (footprint "")
     )
     (path "/cb73e00e-b752-4474-a136-20146bf8e401/5360d48c-d433-4ab9-ab85-b1fcee4d4281"
@@
       (reference "R29") (unit 1) (value "10k") (footprint "Resistor_SMD:R_0603_1608Metric")
     )
+    (path "/8a2d04b1-7a32-450a-8d33-44b6a8475035"
+      (reference "SW1") (unit 1) (value "SW") (footprint "")
+    )
     (path "/8ecd5ebf-2547-4882-86e9-d1153428a5cc/4f4b922b-434d-40d3-bc07-0844c4f27338"
