File: Hardware/Spanner/Spanner/Main.kicad_sch (KiCad schematic)
At the start: 58 parts, among them J1 USB_B_Micro, J2 SWD, J3 MOTOR, J4 MOTOR, J5 MOTOR, J7 Conn_01x02_Male, J8 MOTOR, Q1 BC846, Q3 BC846, Q5 BC846, Q6 BC846, U1 STM32L412K8Tx, U2 USBLC6-2SC6, U3 CURRENT_SENS, U4 RFM95W-868S2, U5 MCP1812AT-033/TT, U6 OPA990

Commit message: softwareproject added
Connections:
- net DI_IN_2 renamed SW_EXT
Changed lines of the file:
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@@
     )
   )
-  (global_label "DI_IN_2" (shape input) (at 43.18 96.52 180) (fields_autoplaced)
+  (global_label "SW_EXT" (shape input) (at 43.18 96.52 180) (fields_autoplaced)
     (effects (font (size 1.27 1.27)) (justify right))
-    (property "Intersheet References" "${INTERSHEET_REFS}" (id 0) (at 33.8121 96.5994 0)
+    (property "Intersheet References" "${INTERSHEET_REFS}" (id 0) (at 33.8121 96.4406 0)
       (effects (font (size 1.27 1.27)) (justify right) hide)
     )
@@
     )
   )
-  (global_label "DI_IN_2" (shape input) (at 210.82 97.79 0) (fields_autoplaced)
+  (global_label "SW_EXT" (shape input) (at 210.82 97.79 0) (fields_autoplaced)
     (effects (font (size 1.27 1.27)) (justify left))
     (property "Intersheet References" "${INTERSHEET_REFS}" (id 0) (at 220.1879 97.7106 0)

Commit message: Update various modules
Parts:
- removed J7: Conn_01x02_Male, Connector_PinHeader_2.54mm:PinHeader_1x02_P2.54mm_Vertical, symbol Connector:Conn_01x02_Male
- added D7: SD0603, Diode_SMD:D_0603_1608Metric, symbol Device:D_Schottky
Connections:
- net VBUS: now also D7.2 (A)
- net at C3.1, D2.1 (K), U5.2 (IN): now also D7.1 (K)
Other:
- moved on the sheet: D2
Changed lines of the file:
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@@
   (junction (at 35.56 63.5) (diameter 0) (color 0 0 0 0)
   )
+  (junction (at 166.37 34.29) (diameter 0) (color 0 0 0 0)
+  )
   (junction (at 236.22 57.15) (diameter 0) (color 0 0 0 0)
   )
@@
   )
   (junction (at 189.23 97.79) (diameter 0) (color 0 0 0 0)
-  )
-  (junction (at 166.37 34.29) (diameter 0) (color 0 0 0 0)
   )
   (junction (at 31.75 149.86) (diameter 0) (color 0 0 0 0)
@@
     (stroke (width 0) (type default) (color 0 0 0 0))
   )
-  (wire (pts (xy 30.48 177.8) (xy 29.21 177.8))
+  (wire (pts (xy 157.48 34.29) (xy 166.37 34.29))
     (stroke (width 0) (type default) (color 0 0 0 0))
   )
@@
     (stroke (width 0) (type default) (color 0 0 0 0))
   )
+  (wire (pts (xy 166.37 20.32) (xy 166.37 22.86))
+    (stroke (width 0) (type default) (color 0 0 0 0))
+  )
   (wire (pts (xy 48.26 153.67) (xy 48.26 152.4))
     (stroke (width 0) (type default) (color 0 0 0 0))
@@
     (stroke (width 0) (type default) (color 0 0 0 0))
   )
-  (wire (pts (xy 166.37 31.115) (xy 166.37 34.29))
-    (stroke (width 0) (type default) (color 0 0 0 0))
-  )
   (wire (pts (xy 134.62 148.59) (xy 134.62 147.32))
     (stroke (width 0) (type default) (color 0 0 0 0))
@@
     (stroke (width 0) (type default) (color 0 0 0 0))
   )
+  (wire (pts (xy 157.48 30.48) (xy 157.48 34.29))
+    (stroke (width 0) (type default) (color 0 0 0 0))
+  )
   (wire (pts (xy 252.73 97.79) (xy 252.73 99.06))
     (stroke (width 0) (type default) (color 0 0 0 0))
@@
     (stroke (width 0) (type default) (color 0 0 0 0))
   )
+  (wire (pts (xy 157.48 20.32) (xy 157.48 22.86))
+    (stroke (width 0) (type default) (color 0 0 0 0))
+  )
   (wire (pts (xy 41.91 114.3) (xy 41.91 113.03))
     (stroke (width 0) (type default) (color 0 0 0 0))
@@
     (stroke (width 0) (type default) (color 0 0 0 0))
   )
-  (wire (pts (xy 30.48 180.34) (xy 30.48 181.61))
-    (stroke (width 0) (type default) (color 0 0 0 0))
-  )
   (wire (pts (xy 236.22 57.15) (xy 238.76 57.15))
     (stroke (width 0) (type default) (color 0 0 0 0))
@@
     (stroke (width 0) (type default) (color 0 0 0 0))
   )
+  (wire (pts (xy 166.37 30.48) (xy 166.37 34.29))
+    (stroke (width 0) (type default) (color 0 0 0 0))
+  )
   (wire (pts (xy 91.44 96.52) (xy 92.71 96.52))
     (stroke (width 0) (type default) (color 0 0 0 0))
@@
     (stroke (width 0) (type default) (color 0 0 0 0))
   )
-  (wire (pts (xy 166.37 20.32) (xy 166.37 23.495))
-    (stroke (width 0) (type default) (color 0 0 0 0))
-  )
   (wire (pts (xy 71.12 88.9) (xy 74.93 88.9))
     (stroke (width 0) (type default) (color 0 0 0 0))
@@
     (stroke (width 0) (type default) (color 0 0 0 0))
   )
-  (wire (pts (xy 30.48 172.72) (xy 30.48 177.8))
-    (stroke (width 0) (type default) (color 0 0 0 0))
-  )
   (wire (pts (xy 29.21 148.59) (xy 29.21 149.86))
     (stroke (width 0) (type default) (color 0 0 0 0))
@@
   )
   (wire (pts (xy 88.9 129.54) (xy 88.9 130.81))
-    (stroke (width 0) (type default) (color 0 0 0 0))
-  )
-  (wire (pts (xy 29.21 180.34) (xy 30.48 180.34))
     (stroke (width 0) (type default) (color 0 0 0 0))
   )
@@
     (pin "1")
   )
-  (symbol (lib_id "Device:D_Schottky") (at 166.37 27.305 90) (unit 1)
-    (in_bom yes) (on_board yes)
-    (property "Reference" "D2" (id 0) (at 171.8564 27.305 0))
-    (property "Value" "SD0603" (id 1) (at 169.545 27.305 0))
-    (property "Footprint" "Diode_SMD:D_0603_1608Metric" (id 2) (at 166.37 27.305 0)
-      (effects (font (size 1.27 1.27)) hide)
-    )
-    (property "Datasheet" "https://www.mouser.ch/datasheet/2/40/schottky-776407.pdf" (id 3) (at 166.37 27.305 0)
-      (effects (font (size 1.27 1.27)) hide)
-    )
-    (property "Hersteller Nr." "SD0603S040S0R2" (id 4) (at 166.37 27.305 90)
-      (effects (font (size 1.27 1.27)) hide)
-    )
-    (property "Mouser Nr." "581-SD0603S040S0R2 " (id 5) (at 166.37 27.305 90)
+  (symbol (lib_id "Device:D_Schottky") (at 166.37 26.67 90) (unit 1)
+    (in_bom yes) (on_board yes)
+    (property "Reference" "D2" (id 0) (at 171.8564 26.67 0))
+    (property "Value" "SD0603" (id 1) (at 169.545 26.67 0))
+    (property "Footprint" "Diode_SMD:D_0603_1608Metric" (id 2) (at 166.37 26.67 0)
+      (effects (font (size 1.27 1.27)) hide)
+    )
+    (property "Datasheet" "https://www.mouser.ch/datasheet/2/40/schottky-776407.pdf" (id 3) (at 166.37 26.67 0)
+      (effects (font (size 1.27 1.27)) hide)
+    )
+    (property "Hersteller Nr." "SD0603S040S0R2" (id 4) (at 166.37 26.67 90)
+      (effects (font (size 1.27 1.27)) hide)
+    )
+    (property "Mouser Nr." "581-SD0603S040S0R2 " (id 5) (at 166.37 26.67 90)
       (effects (font (size 1.27 1.27)) hide)
     )
@@
     (pin "1")
   )
+  (symbol (lib_id "Device:D_Schottky") (at 157.48 26.67 90) (unit 1)
+    (in_bom yes) (on_board yes)
+    (property "Reference" "D7" (id 0) (at 162.9664 26.67 0))
+    (property "Value" "SD0603" (id 1) (at 160.655 26.67 0))
+    (property "Footprint" "Diode_SMD:D_0603_1608Metric" (id 2) (at 157.48 26.67 0)
+      (effects (font (size 1.27 1.27)) hide)
+    )
+    (property "Datasheet" "https://www.mouser.ch/datasheet/2/40/schottky-776407.pdf" (id 3) (at 157.48 26.67 0)
+      (effects (font (size 1.27 1.27)) hide)
+    )
+    (property "Hersteller Nr." "SD0603S040S0R2" (id 4) (at 157.48 26.67 90)
+      (effects (font (size 1.27 1.27)) hide)
+    )
+    (property "Mouser Nr." "581-SD0603S040S0R2 " (id 5) (at 157.48 26.67 90)
+      (effects (font (size 1.27 1.27)) hide)
+    )
+    (pin "1")
+    (pin "2")
+  )
   (symbol (lib_id "Device:R") (at 132.08 38.1 0) (mirror y) (unit 1)
     (in_bom yes) (on_board yes)
@@
     (pin "2")
   )
-  (symbol (lib_id "power:GND") (at 30.48 181.61 0) (unit 1)
-    (in_bom yes) (on_board yes) (fields_autoplaced)
-    (property "Reference" "#PWR0153" (id 0) (at 30.48 187.96 0)
-      (effects (font (size 1.27 1.27)) hide)
-    )
-    (property "Value" "GND" (id 1) (at 30.48 186.69 0))
-    (property "Footprint" "" (id 2) (at 30.48 181.61 0)
-      (effects (font (size 1.27 1.27)) hide)
-    )
-    (property "Datasheet" "" (id 3) (at 30.48 181.61 0)
-      (effects (font (size 1.27 1.27)) hide)
-    )
-    (pin "1")
-  )
   (symbol (lib_id "power:GND") (at 252.73 109.22 0) (unit 1)
     (in_bom yes) (on_board yes)
@@
     (pin "1")
     (pin "2")
+  )
+  (symbol (lib_id "power:VBUS") (at 157.48 20.32 0) (unit 1)
+    (in_bom yes) (on_board yes)
+    (property "Reference" "#PWR0128" (id 0) (at 157.48 24.13 0)
+      (effects (font (size 1.27 1.27)) hide)
+    )
+    (property "Value" "VBUS" (id 1) (at 157.861 15.9258 0))
+    (property "Footprint" "" (id 2) (at 157.48 20.32 0)
+      (effects (font (size 1.27 1.27)) hide)
+    )
+    (property "Datasheet" "" (id 3) (at 157.48 20.32 0)
+      (effects (font (size 1.27 1.27)) hide)
+    )
+    (pin "1")
   )
   (symbol (lib_id "Power_Protection:USBLC6-2SC6") (at 88.9 140.97 0) (unit 1)
@@
       (effects (font (size 1.27 1.27)) hide)
     )
-    (pin "1")
-  )
-  (symbol (lib_id "Connector:Conn_01x02_Male") (at 24.13 177.8 0) (unit 1)
-    (in_bom yes) (on_board yes) (fields_autoplaced)
-    (property "Reference" "J7" (id 0) (at 24.765 172.72 0))
-    (property "Value" "Conn_01x02_Male" (id 1) (at 24.765 175.26 0))
-    (property "Footprint" "Connector_PinHeader_2.54mm:PinHeader_1x02_P2.54mm_Vertical" (id 2) (at 24.13 177.8 0)
-      (effects (font (size 1.27 1.27)) hide)
-    )
-    (property "Datasheet" "~" (id 3) (at 24.13 177.8 0)
-      (effects (font (size 1.27 1.27)) hide)
-    )
-    (pin "1")
-    (pin "2")
-  )
-  (symbol (lib_id "power:+5V") (at 30.48 172.72 0) (unit 1)
-    (in_bom yes) (on_board yes) (fields_autoplaced)
-    (property "Reference" "#PWR0154" (id 0) (at 30.48 176.53 0)
-      (effects (font (size 1.27 1.27)) hide)
-    )
-    (property "Value" "+5V" (id 1) (at 30.48 167.005 0))
-    (property "Footprint" "" (id 2) (at 30.48 172.72 0)
-      (effects (font (size 1.27 1.27)) hide)
-    )
-    (property "Datasheet" "" (id 3) (at 30.48 172.72 0)
-      (effects (font (size 1.27 1.27)) hide)
-    )

Commit message: update spanner
Connections:
- net PWM_2: now also U1.26 (PB3); no longer U1.15 (PB1)
- net SPI_MISO: now also U4.2 (MISO); no longer U4.3 (MOSI)
- net SPI_MOSI: now also U4.3 (MOSI); no longer U4.2 (MISO)
- net VUSB: now also U1.15 (PB1); no longer U1.26 (PB3)
Changed lines of the file:
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@@
     )
   )
-  (global_label "SPI_MISO" (shape output) (at 220.98 35.56 180) (fields_autoplaced)
-    (effects (font (size 1.27 1.27)) (justify right))
-    (property "Intersheet References" "${INTERSHEET_REFS}" (id 0) (at -1.27 -8.89 0)
+  (global_label "SPI_MISO" (shape output) (at 220.98 38.1 180) (fields_autoplaced)
+    (effects (font (size 1.27 1.27)) (justify right))
+    (property "Intersheet References" "${INTERSHEET_REFS}" (id 0) (at -1.27 -6.35 0)
       (effects (font (size 1.27 1.27)) hide)
     )
@@
     )
   )
-  (global_label "VUSB" (shape input) (at 43.18 91.44 180) (fields_autoplaced)
-    (effects (font (size 1.27 1.27)) (justify right))
-    (property "Intersheet References" "${INTERSHEET_REFS}" (id 0) (at 35.8683 91.5194 0)
+  (global_label "VUSB" (shape input) (at 43.18 88.9 180) (fields_autoplaced)
+    (effects (font (size 1.27 1.27)) (justify right))
+    (property "Intersheet References" "${INTERSHEET_REFS}" (id 0) (at 35.8683 88.9794 0)
       (effects (font (size 1.27 1.27)) (justify right) hide)
     )
@@
     )
   )
-  (global_label "SPI_MOSI" (shape input) (at 220.98 38.1 180) (fields_autoplaced)
-    (effects (font (size 1.27 1.27)) (justify right))
-    (property "Intersheet References" "${INTERSHEET_REFS}" (id 0) (at -1.27 -8.89 0)
+  (global_label "SPI_MOSI" (shape input) (at 220.98 35.56 180) (fields_autoplaced)
+    (effects (font (size 1.27 1.27)) (justify right))
+    (property "Intersheet References" "${INTERSHEET_REFS}" (id 0) (at -1.27 -11.43 0)
       (effects (font (size 1.27 1.27)) hide)
     )
@@
     )
   )
-  (global_label "PWM_2" (shape input) (at 43.18 88.9 180) (fields_autoplaced)
-    (effects (font (size 1.27 1.27)) (justify right))
-    (property "Intersheet References" "${INTERSHEET_REFS}" (id 0) (at 34.4169 88.8206 0)
-      (effects (font (size 1.27 1.27)) (justify right) hide)
-    )
+  (global_label "PWM_2" (shape input) (at 43.18 91.44 180) (fields_autoplaced)
+    (effects (font (size 1.27 1.27)) (justify right))
+    (property "Intersheet References" "${INTERSHEET_REFS}" (id 0) (at 34.4169 91.3606 0)
+      (effects (font (size 1.27 1.27)) (justify right) hide)
+    )

Commit message: FW update
Parts:
- removed R21: 10k, Resistor_SMD:R_0603_1608Metric, symbol Device:R
Changed lines of the file:
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@@
   (junction (at 48.26 143.51) (diameter 0) (color 0 0 0 0)
-  )
-  (junction (at 261.62 82.55) (diameter 0) (color 0 0 0 0)
   )
   (junction (at 236.22 22.86) (diameter 0) (color 0 0 0 0)
@@
     (stroke (width 0) (type default) (color 0 0 0 0))
   )
-  (wire (pts (xy 261.62 81.28) (xy 261.62 82.55))
-    (stroke (width 0) (type default) (color 0 0 0 0))
-  )
   (wire (pts (xy 195.58 49.53) (xy 195.58 48.26))
     (stroke (width 0) (type default) (color 0 0 0 0))
@@
   )
   (wire (pts (xy 64.77 31.75) (xy 63.5 31.75))
-    (stroke (width 0) (type default) (color 0 0 0 0))
-  )
-  (wire (pts (xy 261.62 72.39) (xy 261.62 73.66))
     (stroke (width 0) (type default) (color 0 0 0 0))
   )
@@
     (pin "2")
   )
-  (symbol (lib_id "power:+24V") (at 261.62 72.39 0) (unit 1)
-    (in_bom yes) (on_board yes) (fields_autoplaced)
-    (property "Reference" "#PWR0150" (id 0) (at 261.62 76.2 0)
-      (effects (font (size 1.27 1.27)) hide)
-    )
-    (property "Value" "+24V" (id 1) (at 261.62 67.31 0))
-    (property "Footprint" "" (id 2) (at 261.62 72.39 0)
-      (effects (font (size 1.27 1.27)) hide)
-    )
-    (property "Datasheet" "" (id 3) (at 261.62 72.39 0)
-      (effects (font (size 1.27 1.27)) hide)
-    )
-    (pin "1")
-  )
   (symbol (lib_id "power:GND") (at 88.9 152.4 0) (unit 1)
     (in_bom yes) (on_board yes)
@@
     (pin "1")
   )
-  (symbol (lib_id "Device:R") (at 261.62 77.47 0) (mirror y) (unit 1)
-    (in_bom yes) (on_board yes)
-    (property "Reference" "R21" (id 0) (at 266.8778 77.47 90))
-    (property "Value" "10k" (id 1) (at 264.5664 77.47 90))
-    (property "Footprint" "Resistor_SMD:R_0603_1608Metric" (id 2) (at 263.398 77.47 90)
-      (effects (font (size 1.27 1.27)) hide)
-    )
-    (property "Datasheet" "" (id 3) (at 261.62 77.47 0)
-      (effects (font (size 1.27 1.27)) hide)
-    )
-    (property "Hersteller Nr." "RT0603FRE0710KL" (id 4) (at 261.62 77.47 0)
-      (effects (font (size 1.27 1.27)) hide)
-    )
-    (property "Mouser Nr." "603-RT0603FRE0710KL" (id 5) (at 261.62 77.47 0)
-      (effects (font (size 1.27 1.27)) hide)
-    )
-    (pin "1")
-    (pin "2")
-  )
   (symbol (lib_id "power:GND") (at 252.73 109.22 0) (unit 1)

Commit message: software stabilisation
Parts:
- R28: value 10k -> 1.7k; Hersteller Nr. RT0603FRE0710KL -> (none); Mouser Nr. 603-RT0603FRE0710KL -> (none)
- R29: value 10k -> 3.3k; Hersteller Nr. RT0603FRE0710KL -> (none); Mouser Nr. 603-RT0603FRE0710KL -> (none)
Other:
- moved on the sheet: R25

Commit message: update firmware
Connections:
- net PWM_1 renamed PWM_SPEED
- net PWM_2 renamed PWM_DIRECTION
Changed lines of the file:
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@@
     )
   )
-  (global_label "PWM_1" (shape input) (at 182.88 147.32 180) (fields_autoplaced)
-    (effects (font (size 1.27 1.27)) (justify right))
-    (property "Intersheetrefs" "${INTERSHEET_REFS}" (at 174.1169 147.2406 0)
+  (global_label "PWM_SPEED" (shape input) (at 182.88 147.32 180) (fields_autoplaced)
+    (effects (font (size 1.27 1.27)) (justify right))
+    (property "Intersheetrefs" "${INTERSHEET_REFS}" (at 168.7863 147.32 0)
       (effects (font (size 1.27 1.27)) (justify right) hide)
     )
@@
     )
   )
-  (global_label "PWM_2" (shape input) (at 232.41 147.32 180) (fields_autoplaced)
-    (effects (font (size 1.27 1.27)) (justify right))
-    (property "Intersheetrefs" "${INTERSHEET_REFS}" (at 223.6469 147.2406 0)
+  (global_label "PWM_DIRECTION" (shape input) (at 232.41 147.32 180) (fields_autoplaced)
+    (effects (font (size 1.27 1.27)) (justify right))
+    (property "Intersheetrefs" "${INTERSHEET_REFS}" (at 214.5666 147.32 0)
       (effects (font (size 1.27 1.27)) (justify right) hide)
     )
@@
     )
   )
-  (global_label "PWM_2" (shape input) (at 43.18 91.44 180) (fields_autoplaced)
-    (effects (font (size 1.27 1.27)) (justify right))
-    (property "Intersheetrefs" "${INTERSHEET_REFS}" (at 34.4169 91.3606 0)
+  (global_label "PWM_DIRECTION" (shape input) (at 43.18 91.44 180) (fields_autoplaced)
+    (effects (font (size 1.27 1.27)) (justify right))
+    (property "Intersheetrefs" "${INTERSHEET_REFS}" (at 25.3366 91.44 0)
       (effects (font (size 1.27 1.27)) (justify right) hide)
     )
@@
     )
   )
-  (global_label "PWM_1" (shape input) (at 73.66 104.14 0) (fields_autoplaced)
-    (effects (font (size 1.27 1.27)) (justify left))
-    (property "Intersheetrefs" "${INTERSHEET_REFS}" (at 82.4231 104.0606 0)
-      (effects (font (size 1.27 1.27)) (justify left) hide)
-    )
+  (global_label "PWM_SPEED" (shape input) (at 73.66 104.14 0) (fields_autoplaced)
+    (effects (font (size 1.27 1.27)) (justify left))
+    (property "Intersheetrefs" "${INTERSHEET_REFS}" (at 87.7537 104.14 0)
+      (effects (font (size 1.27 1.27)) (justify left) hide)
+    )
