File: Hardware/Cobot/Cobot/Cobot.kicad_pcb (KiCad board)
At the start: 2 copper layers, 78 x 52.5 mm, 170 parts, among them J1 USB_B_Micro, J2 Conn_02x02_Counter_Clockwise, J3 DO, J4 DAC, J5 DI, J6 ADC, J7 Power, Q1 SI7309D, U1 STM32L433RCTxP, U2 USBLC6-2SC6, U3 RFM95W-868S2, U4 AP63203WU, U5 OPA990, U6 OPA990

Commit message: Software implementation
Parts:
- added R88: 100k, Resistor_SMD:R_0603_1608Metric, F.Cu at (128.5, 140.5)
- moved J4 2.54 mm to (106.0, 165.0), turned to 0 degrees
- moved J6 2.54 mm to (99.9, 129.8), turned to 180 degrees
- moved J7 2.54 mm to (107.7, 129.8), turned to 180 degrees
Connections:
- J4 pad 1: DAC_OUT_2 -> DAC_OUT_1
- J4 pad 2: DAC_OUT_1 -> DAC_OUT_2
- J6 pad 1: ADC_IN_1 -> ADC_IN_2
- J6 pad 2: ADC_IN_2 -> ADC_IN_1
- J7 pad 1: GND -> VCC
- J7 pad 2: VCC -> GND
- U1 pad 30: +3.3V -> unconnected-(U1-Pad30)
- U1 pad 52: SPI_MOSI -> SPI_MISO
- U1 pad 53: SPI_MISO -> SPI_MOSI
- U1 pad 59: unconnected-(U1-Pad59) -> Net-(R88-Pad2)
- U1 pad 62: +3.3V -> unconnected-(U1-Pad62)
Routing:
- net Net-(R88-Pad2): track 0.00 -> 10.1 mm
- net SPI_MISO: track 13.3 -> 17.4 mm
- net SPI_MOSI: track 11.2 -> 15.3 mm
- net +3.3V: track 133.1 -> 129.1 mm
- net VUSB: track 26.5 -> 27.8 mm
- net SPI_SCK: track 18.4 -> 19.7 mm

Commit message: Update Firmware
Connections:
- U1 pad 17: unconnected-(U1-Pad17) -> VUSB
- U1 pad 48: VUSB -> +3.3V
Routing:
- net VUSB: track 27.8 -> 48.3 mm
- net +3.3V: track 129.1 -> 132.6 mm, vias 9 -> 10
- net GND: track 181.0 -> 183.2 mm, vias 80 -> 81
- net SWDIO: track 11.0 -> 10.4 mm

Commit message: Update HW and SW
Parts:
- moved J2 63.8 mm to (172.7, 120.9)
- moved C1 63.8 mm to (156.9, 98.4)
- moved C11 63.8 mm to (152.9, 92.5)
- moved C17 63.8 mm to (158.9, 85.6)
- moved F2 63.8 mm to (131.1, 112.7)
- moved F3 63.8 mm to (114.8, 103.6)
- moved F4 63.8 mm to (132.8, 103.6)
- moved F6 63.8 mm to (140.1, 112.7)
- moved F8 63.8 mm to (141.8, 103.6)
- moved H2 63.8 mm to (113.9, 124.4)
- moved H3 63.8 mm to (113.9, 78.9)
- moved J3 63.8 mm to (120.5, 119.1)
- moved J4 63.8 mm to (150.4, 119.1)
- moved J5 63.8 mm to (137.3, 83.9)
- moved J6 63.8 mm to (144.3, 83.9)
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Connections:
- U3 pad 2: SPI_MOSI -> SPI_MISO
- U3 pad 3: SPI_MISO -> SPI_MOSI
Routing:
- net SPI_MISO: track 17.4 -> 11.6 mm
- net SPI_MOSI: track 15.3 -> 13.5 mm
- net SPI_SCK: track 19.7 -> 18.2 mm
Other:
- outline, holes or cut-outs redrawn
