File: Hardware/Cobot/Cobot/Connection.kicad_sch (KiCad schematic)
At the start: 9 parts, among them J3 DO, J4 DAC, J5 DI, J6 ADC, J7 Power

Commit message: Software implementation
Connections:
- net ADC_IN_1: now also J6.2 (Pin_2); no longer J6.1 (Pin_1)
- net ADC_IN_2: now also J6.1 (Pin_1); no longer J6.2 (Pin_2)
- net DAC_OUT_1: now also J4.1 (Pin_1); no longer J4.2 (Pin_2)
- net DAC_OUT_2: now also J4.2 (Pin_2); no longer J4.1 (Pin_1)
- net GND: now also J7.2 (Pin_2); no longer J7.1 (Pin_1)
- net VCC: now also J7.1 (Pin_1); no longer J7.2 (Pin_2)
Changed lines of the file:
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@@
     )
   )
-  (symbol (lib_id "Connector:Screw_Terminal_01x02") (at 165.1 59.69 0) (mirror x) (unit 1)
+  (symbol (lib_id "Connector:Screw_Terminal_01x02") (at 165.1 57.15 0) (unit 1)
     (in_bom yes) (on_board yes) (fields_autoplaced)
-    (property "Reference" "J7" (id 0) (at 165.1 50.8 0))
-    (property "Value" "Power" (id 1) (at 165.1 53.34 0))
-    (property "Footprint" "MK_Footprints:TerminalBlock_Phoenix_MPT-0,5-2-2.54_1x02_P2.54mm_Horizontal" (id 2) (at 165.1 59.69 0)
+    (property "Reference" "J7" (id 0) (at 167.64 57.1499 0)
+      (effects (font (size 1.27 1.27)) (justify left))
+    )
+    (property "Value" "Power" (id 1) (at 167.64 59.6899 0)
+      (effects (font (size 1.27 1.27)) (justify left))
+    )
+    (property "Footprint" "MK_Footprints:TerminalBlock_Phoenix_MPT-0,5-2-2.54_1x02_P2.54mm_Horizontal" (id 2) (at 165.1 57.15 0)
       (effects (font (size 1.27 1.27)) hide)
     )
-    (property "Datasheet" "~" (id 3) (at 165.1 59.69 0)
+    (property "Datasheet" "~" (id 3) (at 165.1 57.15 0)
       (effects (font (size 1.27 1.27)) hide)
     )
@@
     (pin "8")
   )
-  (symbol (lib_id "Connector:Screw_Terminal_01x02") (at 88.9 68.58 0) (unit 1)
+  (symbol (lib_id "Connector:Screw_Terminal_01x02") (at 88.9 71.12 0) (mirror x) (unit 1)
     (in_bom yes) (on_board yes) (fields_autoplaced)
-    (property "Reference" "J4" (id 0) (at 91.44 68.5799 0)
-      (effects (font (size 1.27 1.27)) (justify left))
-    )
-    (property "Value" "DAC" (id 1) (at 91.44 71.1199 0)
-      (effects (font (size 1.27 1.27)) (justify left))
-    )
-    (property "Footprint" "MK_Footprints:TerminalBlock_Phoenix_MPT-0,5-2-2.54_1x02_P2.54mm_Horizontal" (id 2) (at 88.9 68.58 0)
+    (property "Reference" "J4" (id 0) (at 88.9 62.23 0))
+    (property "Value" "DAC" (id 1) (at 88.9 64.77 0))
+    (property "Footprint" "MK_Footprints:TerminalBlock_Phoenix_MPT-0,5-2-2.54_1x02_P2.54mm_Horizontal" (id 2) (at 88.9 71.12 0)
       (effects (font (size 1.27 1.27)) hide)
     )
-    (property "Datasheet" "~" (id 3) (at 88.9 68.58 0)
+    (property "Datasheet" "~" (id 3) (at 88.9 71.12 0)
       (effects (font (size 1.27 1.27)) hide)
     )
@@
     (pin "8")
   )
-  (symbol (lib_id "Connector:Screw_Terminal_01x02") (at 134.62 67.31 0) (unit 1)
+  (symbol (lib_id "Connector:Screw_Terminal_01x02") (at 134.62 69.85 0) (mirror x) (unit 1)
     (in_bom yes) (on_board yes) (fields_autoplaced)
-    (property "Reference" "J6" (id 0) (at 137.16 67.3099 0)
-      (effects (font (size 1.27 1.27)) (justify left))
-    )
-    (property "Value" "ADC" (id 1) (at 137.16 69.8499 0)
-      (effects (font (size 1.27 1.27)) (justify left))
-    )
-    (property "Footprint" "MK_Footprints:TerminalBlock_Phoenix_MPT-0,5-2-2.54_1x02_P2.54mm_Horizontal" (id 2) (at 134.62 67.31 0)
+    (property "Reference" "J6" (id 0) (at 134.62 60.96 0))
+    (property "Value" "ADC" (id 1) (at 134.62 63.5 0))
+    (property "Footprint" "MK_Footprints:TerminalBlock_Phoenix_MPT-0,5-2-2.54_1x02_P2.54mm_Horizontal" (id 2) (at 134.62 69.85 0)
       (effects (font (size 1.27 1.27)) hide)
     )
-    (property "Datasheet" "~" (id 3) (at 134.62 67.31 0)
+    (property "Datasheet" "~" (id 3) (at 134.62 69.85 0)
       (effects (font (size 1.27 1.27)) hide)
     )
